Commit message: change the args of the control mode

File: urdf/sciurus17.urdf.xacro (robot description, xacro)
@@ -19,34 +19,40 @@
   <xacro:arg name="load_trans2" default="false" />
   <xacro:arg name="load_trans3" default="false" />
-  <xacro:arg name="use_effort_right_arm" default="false" />
-  <xacro:property name="right_arm_interface" value="position"/>
-  <xacro:if value="$(arg use_effort_right_arm)">
-    <xacro:property name="right_arm_interface" value="effort"/>
-  </xacro:if>
-  <xacro:arg name="use_effort_left_wrist" default="false" />
-  <xacro:property name="left_wrist_interface" value="position"/>
-  <xacro:if value="$(arg use_effort_left_wrist)">
-    <xacro:property name="left_wrist_interface" value="effort"/>
-  </xacro:if>
+  <xacro:arg name="right_arm_interface" default="position" />
+  <xacro:arg name="left_arm_interface" default="position" />
   <xacro:if value="$(arg use_gazebo_simulation)">
     <xacro:include filename="$(find sciurus17_description)/urdf/sciurus17_gazebo.xacro"/>
     <xacro:if value="$(arg load_trans1)">
-      <xacro:default_transmission joint_name="r_arm_joint1" interface="${right_arm_interface}"/>
-      <xacro:default_transmission joint_name="r_arm_joint2" interface="${right_arm_interface}"/>
-      <xacro:default_transmission joint_name="r_arm_joint3" interface="${right_arm_interface}"/>
-      <xacro:default_transmission joint_name="r_arm_joint4" interface="${right_arm_interface}"/>
-      <xacro:default_transmission joint_name="r_arm_joint5" interface="${right_arm_interface}"/>
-      <xacro:default_transmission joint_name="r_arm_joint6" interface="${right_arm_interface}"/>
-      <xacro:default_transmission joint_name="r_arm_joint7" interface="${right_arm_interface}"/>
+      <xacro:default_transmission joint_name="r_arm_joint1"
+                                  interface="$(arg right_arm_interface)"/>
+      <xacro:default_transmission joint_name="r_arm_joint2"
+                                  interface="$(arg right_arm_interface)"/>
+      <xacro:default_transmission joint_name="r_arm_joint3"
+                                  interface="$(arg right_arm_interface)"/>
+      <xacro:default_transmission joint_name="r_arm_joint4"
+                                  interface="$(arg right_arm_interface)"/>
+      <xacro:default_transmission joint_name="r_arm_joint5"
+                                  interface="$(arg right_arm_interface)"/>
+      <xacro:default_transmission joint_name="r_arm_joint6"
+                                  interface="$(arg right_arm_interface)"/>
+      <xacro:default_transmission joint_name="r_arm_joint7"
+                                  interface="$(arg right_arm_interface)"/>
       <xacro:default_transmission joint_name="r_hand_joint"/>
     </xacro:if>
     <xacro:if value="$(arg load_trans2)">
-      <xacro:default_transmission joint_name="l_arm_joint1"/>
-      <xacro:default_transmission joint_name="l_arm_joint2"/>
-      <xacro:default_transmission joint_name="l_arm_joint3"/>
-      <xacro:default_transmission joint_name="l_arm_joint4"/>
-      <xacro:default_transmission joint_name="l_arm_joint5"/>
-      <xacro:default_transmission joint_name="l_arm_joint6"/>
-      <xacro:default_transmission joint_name="l_arm_joint7" interface="${left_wrist_interface}"/>
+      <xacro:default_transmission joint_name="l_arm_joint1"
+                                  interface="$(arg left_arm_interface)"/>
+      <xacro:default_transmission joint_name="l_arm_joint2"
+                                  interface="$(arg left_arm_interface)"/>
+      <xacro:default_transmission joint_name="l_arm_joint3"
+                                  interface="$(arg left_arm_interface)"/>
+      <xacro:default_transmission joint_name="l_arm_joint4"
+                                  interface="$(arg left_arm_interface)"/>
+      <xacro:default_transmission joint_name="l_arm_joint5"
+                                  interface="$(arg left_arm_interface)"/>
+      <xacro:default_transmission joint_name="l_arm_joint6"
+                                  interface="$(arg left_arm_interface)"/>
+      <xacro:default_transmission joint_name="l_arm_joint7"
+                                  interface="$(arg left_arm_interface)"/>
       <xacro:default_transmission joint_name="l_hand_joint"/>
     </xacro:if>

File: urdf/sciurus17_right_arm.xacro (robot description, xacro)
@@ -100,12 +100,12 @@
         <origin rpy="1.5708 0 0" xyz="0.0 0.0 0.0"/>
         <geometry>
-          <mesh filename="package://sciurus17_description/meshes/visual/L_Link3.stl" scale="1.0 -1.0 1.0"/>
-        </geometry>
-        <material name="${arm_color}"/>
-      </visual>
-      <collision>
-        <origin rpy="1.5708 0 0" xyz="0.0 0.0 0.0"/>
-        <geometry>
-          <mesh filename="package://sciurus17_description/meshes/collision/L_Link3.stl" scale="1.0 -1.0 1.0"/>
+          <mesh filename="package://sciurus17_description/meshes/visual/R_Link3.stl" scale="1.0 -1.0 1.0"/>
+        </geometry>
+        <material name="${arm_color}"/>
+      </visual>
+      <collision>
+        <origin rpy="1.5708 0 0" xyz="0.0 0.0 0.0"/>
+        <geometry>
+          <mesh filename="package://sciurus17_description/meshes/collision/R_Link3.stl" scale="1.0 -1.0 1.0"/>
         </geometry>
       </collision>
